File: IC_CLOCK_POWER/IC_CLOCK_POWER.kicad_sch (KiCad schematic)
At the start: 24 parts, among them J1 Conn_01x02_Pin, J2 Conn_01x04_Pin, U1 LM7805_TO220, U2 LM317T

Commit message: Fixing schematic ..and footprints
Parts:
- removed U1: LM7805_TO220, Package_TO_SOT_THT:TO-220-3_Vertical, symbol Regulator_Linear:LM7805_TO220
- added U1: LM7805_TO220_HEAT_SINK, IC_CLOCK:TO-220-HEADSINK-35X12, symbol IC_CLOCK:LM7805_TO220_HEAT_SINK
- C10: value ${SIM.PARAMS} -> 0.1u
- C4: footprint Resistor_THT:R_Axial_DIN0207_L6.3mm_D2.5mm_P7.62mm_Horizontal -> Capacitor_THT:CP_Radial_D10.0mm_P7.50mm
- C7: footprint Capacitor_THT:CP_Radial_D18.0mm_P7.50mm -> Capacitor_THT:CP_Radial_D10.0mm_P7.50mm
- C9: footprint Capacitor_THT:CP_Axial_L11.0mm_D6.0mm_P18.00mm_Horizontal -> Capacitor_THT:CP_Radial_D5.0mm_P2.50mm
- J2: footprint Connector_PinHeader_2.54mm:PinHeader_1x04_P2.54mm_Horizontal -> Connector_JST:JST_EH_S4B-EH_1x04_P2.50mm_Horizontal
- U2: footprint digikey-footprints:TO-220-3 -> IC_CLOCK:TO-220-HEADSINK-35X12
Connections:
- net +5V: now also U1.3 (VO)
- net GND: now also U1.2 (GND)
- net at C4.1, D4.1 (K), D8.1 (K): now also U1.1 (VI)
- no-connect marks 0 -> 2
Changed lines of the file:
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@@
 	)
 	(junction
+		(at 102.87 35.56)
+		(diameter 0)
+		(color 0 0 0 0)
+	)
+	(junction
 		(at 120.65 101.6)
 		(diameter 0)
@@
 	)
 	(junction
-		(at 100.33 35.56)
-		(diameter 0)
-		(color 0 0 0 0)
-	)
-	(junction
 		(at 120.65 35.56)
 		(diameter 0)
@@
 		(color 0 0 0 0)
 	)
+	(no_connect
+		(at 118.11 104.14)
+	)
+	(no_connect
+		(at 118.11 105.41)
+	)
 	(wire
 		(pts
@@
 	(wire
 		(pts
-			(xy 100.33 35.56) (xy 102.87 35.56)
-		)
-		(stroke
-			(width 0)
-			(type default)
-		)
-	)
-	(wire
-		(pts
-			(xy 100.33 49.53) (xy 102.87 49.53)
-		)
-		(stroke
-			(width 0)
-			(type default)
-		)
-	)
-	(wire
-		(pts
 			(xy 114.3 76.2) (xy 120.65 76.2)
 		)
@@
 	(wire
 		(pts
-			(xy 100.33 35.56) (xy 100.33 49.53)
+			(xy 102.87 35.56) (xy 102.87 49.53)
 		)
 		(stroke
@@
 	(wire
 		(pts
-			(xy 92.71 35.56) (xy 100.33 35.56)
+			(xy 92.71 35.56) (xy 102.87 35.56)
 		)
 		(stroke
@@
 			)
 		)
-		(property "Footprint" "Capacitor_THT:CP_Axial_L11.0mm_D6.0mm_P18.00mm_Horizontal"
+		(property "Footprint" "Capacitor_THT:CP_Radial_D5.0mm_P2.50mm"
 			(at 133.0452 57.15 0)
 			(effects
@@
 			)
 		)
-		(property "Footprint" "Resistor_THT:R_Axial_DIN0207_L6.3mm_D2.5mm_P7.62mm_Horizontal"
+		(property "Footprint" "Capacitor_THT:CP_Radial_D10.0mm_P7.50mm"
 			(at 93.6752 116.84 0)
 			(effects
@@
 			)
 		)
-		(property "Value" "${SIM.PARAMS}"
+		(property "Value" "0.1u"
 			(at 106.68 52.0699 0)
 			(effects
@@
 				)
 				(justify right)
-				(hide yes)
 			)
 		)
@@
 				)
 				(justify right)
+				(hide yes)
 			)
 		)
@@
 			)
 		)
-		(property "Footprint" "digikey-footprints:TO-220-3"
+		(property "Footprint" "IC_CLOCK:TO-220-HEADSINK-35X12"
 			(at 115.57 30.48 0)
 			(effects
@@
 	)
 	(symbol
+		(lib_id "IC_CLOCK:LM7805_TO220_HEAT_SINK")
+		(at 110.49 101.6 0)
+		(unit 1)
+		(exclude_from_sim no)
+		(in_bom yes)
+		(on_board yes)
+		(dnp no)
+		(fields_autoplaced yes)
+		(property "Reference" "U1"
+			(at 110.49 95.25 0)
+			(effects
+				(font
+					(size 1.27 1.27)
+				)
+			)
+		)
+		(property "Value" "LM7805_TO220_HEAT_SINK"
+			(at 110.49 97.79 0)
+			(effects
+				(font
+					(size 1.27 1.27)
+				)
+			)
+		)
+		(property "Footprint" "IC_CLOCK:TO-220-HEADSINK-35X12"
+			(at 110.49 95.885 0)
+			(effects
+				(font
+					(size 1.27 1.27)
+					(italic yes)
+				)
+				(hide yes)
+			)
+		)
+		(property "Datasheet" "https://www.onsemi.cn/PowerSolutions/document/MC7800-D.PDF"
+			(at 110.49 102.87 0)
+			(effects
+				(font
+					(size 1.27 1.27)
+				)
+				(hide yes)
+			)
+		)
+		(property "Description" "Positive 1A 35V Linear Regulator, Fixed Output 5V, TO-220"
+			(at 110.49 101.6 0)
+			(effects
+				(font
+					(size 1.27 1.27)
+				)
+				(hide yes)
+			)
+		)
+		(pin "4"
+		)
+		(pin "1"
+		)
+		(pin "5"
+		)
+		(pin "3"
+		)
+		(pin "2"
+		)
+		(instances
+			(project "IC_CLOCK_POWER"
+				(path "/5e066d53-1ba4-4246-9683-66b64aadc766"
+					(reference "U1")
+					(unit 1)
+				)
+			)
+		)
+	)
+	(symbol
 		(lib_id "power:GND")
 		(at 167.64 63.5 0)
@@
 	)
 	(symbol
-		(lib_id "Regulator_Linear:LM7805_TO220")
-		(at 110.49 101.6 0)
-		(unit 1)
-		(exclude_from_sim no)
-		(in_bom yes)
-		(on_board yes)
-		(dnp no)
-		(fields_autoplaced yes)
-		(property "Reference" "U1"
-			(at 110.49 95.25 0)
-			(effects
-				(font
-					(size 1.27 1.27)
-				)
-			)
-		)
-		(property "Value" "LM7805_TO220"
-			(at 110.49 97.79 0)
-			(effects
-				(font
-					(size 1.27 1.27)
-				)
-			)
-		)
-		(property "Footprint" "Package_TO_SOT_THT:TO-220-3_Vertical"
-			(at 110.49 95.885 0)
-			(effects
-				(font
-					(size 1.27 1.27)
-					(italic yes)
-				)
-				(hide yes)
-			)
-		)
-		(property "Datasheet" "https://www.onsemi.cn/PowerSolutions/document/MC7800-D.PDF"
-			(at 110.49 102.87 0)
-			(effects
-				(font
-					(size 1.27 1.27)
-				)
-				(hide yes)
-			)
-		)
-		(property "Description" "Positive 1A 35V Linear Regulator, Fixed Output 5V, TO-220"
-			(at 110.49 101.6 0)
-			(effects
-				(font
-					(size 1.27 1.27)
-				)
-				(hide yes)
-			)
-		)
-		(pin "2"
-		)
-		(pin "3"
-		)
-		(pin "1"
-		)
-		(instances
-			(project "IC_CLOCK_POWER"
-				(path "/5e066d53-1ba4-4246-9683-66b64aadc766"
-					(reference "U1")
-					(unit 1)
-				)
-			)
-		)
-	)
-	(symbol
 		(lib_id "Device:C")
 		(at 135.89 113.03 180)
@@
 		(on_board yes)
 		(dnp no)
-		(fields_autoplaced yes)
 		(property "Reference" "D4"
-			(at 95.25 52.0699 90)
+			(at 88.646 52.832 90)
 			(effects
 				(font
@@
 		)
 		(property "Value" "1N4002"
-			(at 95.25 54.6099 90)
+			(at 89.662 50.038 90)
 			(effects
 				(font
@@
 			)
 		)
-		(property "Footprint" "Capacitor_THT:CP_Radial_D18.0mm_P7.50mm"
+		(property "Footprint" "Capacitor_THT:CP_Radial_D10.0mm_P7.50mm"
 			(at 63.1952 67.31 0)
 			(effects
@@
 			)
 		)
-		(property "Footprint" "Connector_PinHeader_2.54mm:PinHeader_1x04_P2.54mm_Horizontal"
+		(property "Footprint" "Connector_JST:JST_EH_S4B-EH_1x04_P2.50mm_Horizontal"
 			(at 208.28 25.4 0)
 			(effects

Commit message: Update to files ...
Parts:
- removed D3: Bridge_Rectifiers, IC_CLOCK:Bridge_Rectifier_4EDIP, symbol IC_CLOCK:Bridge_Rectifiers
- removed U1: LM7805_TO220_HEAT_SINK, IC_CLOCK:TO-220-HEADSINK-35X12, symbol IC_CLOCK:LM7805_TO220_HEAT_SINK
- removed U2: LM317T, IC_CLOCK:TO-220-HEADSINK-35X12, symbol dk_PMIC-Voltage-Regulators-Linear:LM317T
- added D5: DB107, IC_CLOCK:Bridge_Rectifier_4EDIP, symbol IC_CLOCK:Bridge_Rectifiers
- added U1: LM317T, Package_TO_SOT_THT:TO-220F-3_HEATSINK_Vertical, symbol dk_PMIC-Voltage-Regulators-Linear:LM317T
- added U2: L7805, Package_TO_SOT_THT:TO-220F-3_HEATSINK_Vertical, symbol Regulator_Linear:L7805
- C10: value 0.1u -> ${SIM.PARAMS}
- C4: footprint Capacitor_THT:CP_Radial_D10.0mm_P7.50mm -> Resistor_THT:R_Axial_DIN0207_L6.3mm_D2.5mm_P7.62mm_Horizontal
- C7: footprint Capacitor_THT:CP_Radial_D10.0mm_P7.50mm -> Capacitor_THT:CP_Radial_D18.0mm_P7.50mm
- C9: footprint Capacitor_THT:CP_Radial_D5.0mm_P2.50mm -> Capacitor_THT:CP_Axial_L11.0mm_D6.0mm_P18.00mm_Horizontal
- J2: footprint Connector_JST:JST_EH_S4B-EH_1x04_P2.50mm_Horizontal -> Connector_PinHeader_2.54mm:PinHeader_1x04_P2.54mm_Horizontal
Connections:
- net +10V: now also U1.2 (OUT)
- net +5V: now also U2.3 (OUT)
- net 12VAC: now also D5.4
- net GND: now also D5.2 (-), U2.2 (GND)
- net at C9.1, D6.2 (A), R3.1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: now also U1.1 (ADJ)
- net at C4.1, D4.1 (K), D8.1 (K): now also U2.1 (IN)
- net at C10.2, C6.1, C7.1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: now also D5.1 (+), U1.3 (IN)
- net AC-GND: no longer names the net of J1.2 (Pin_2)
- net AC-GND: now also D5.3
- no-connect marks 2 -> 0

Commit message: Fixing schematic ..
Parts:
- removed D5: DB107, IC_CLOCK:Bridge_Rectifier_4EDIP, symbol IC_CLOCK:Bridge_Rectifiers
- removed U1: LM317T, Package_TO_SOT_THT:TO-220F-3_HEATSINK_Vertical, symbol dk_PMIC-Voltage-Regulators-Linear:LM317T
- removed U2: L7805, Package_TO_SOT_THT:TO-220F-3_HEATSINK_Vertical, symbol Regulator_Linear:L7805
- added D3: Bridge_Rectifiers, IC_CLOCK:Bridge_Rectifier_4EDIP, symbol IC_CLOCK:Bridge_Rectifiers
- added U1: LM7805_TO220, Package_TO_SOT_THT:TO-220-3_Vertical, symbol Regulator_Linear:LM7805_TO220
- added U2: LM317T, digikey-footprints:TO-220-3, symbol dk_PMIC-Voltage-Regulators-Linear:LM317T
Connections:
- net +10V: now also U2.2 (OUT)
- net +5V: now also U1.3 (VO)
- net 12VAC: now also D3.4
- net GND: now also D3.2 (-), U1.2 (GND)
- net at C9.1, D6.2 (A), R3.1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: now also U2.1 (ADJ)
- net AC-GND: now reaches J1.2 (Pin_2)
- net AC-GND: now also D3.3
- net at C4.1, D4.1 (K), D8.1 (K): now also U1.1 (VI)
- net at C10.2, C6.1, C7.1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: now also D3.1 (+), U2.3 (IN)
