File: IC_CLOCK_7SEG/IC_CLOCK_7SEGMENT_DISPLAY.kicad_pcb (KiCad board)
At the start: 2 copper layers, 50 x 86 mm, 17 parts, among them J1 Conn_01x08_Pin, U2 4543

Commit message: Adding component ..
Parts:
- removed REF**: M3, MountingHole:MountingHole_3.2mm_M3
- removed REF** (x3): MountingHole_3.2mm_M3, MountingHole:MountingHole_3.2mm_M3
- added J2: Conn_01x03_Pin, Connector_PinHeader_2.54mm:PinHeader_1x03_P2.54mm_Horizontal, B.Cu at (143.1, 92.5)
Routing:
- net +10V: track 41.5 -> 75.6 mm
- net +5V: track 33.4 -> 46.5 mm
Other:
- board text added: "+10v"
- board text added: "+5v"
- board text added: "gnd"
