File: IC_CLOCK_7SEG/IC_CLOCK_7SEGMENT_DISPLAY.kicad_sch (KiCad schematic)
At the start: 13 parts, among them J1 Conn_01x08_Pin, U2 4543

Commit message: Adding component ..
Parts:
- added J2: Conn_01x03_Pin, Connector_PinHeader_2.54mm:PinHeader_1x03_P2.54mm_Horizontal, symbol Connector:Conn_01x03_Pin
Connections:
- net +10V: now also J2.3 (Pin_3)
- net +5V: now also J2.2 (Pin_2)
- net GND: now also J2.1 (Pin_1)
